Commit message: 2022/06/18

File: pick_and_place/urdf/redbox.urdf.xacro (robot description, xacro)
@@ -13,5 +13,5 @@
                 <origin xyz="0.0 0.0 0.0" rpy="0.0 0.0 0.0"/>
                 <geometry>
-                <box size="0.035 0.035 0.06"/>
+                <box size="0.036 0.036 0.06"/>
                 </geometry>
                 <material name="red"/>
@@ -20,5 +20,5 @@
                 <origin xyz="0.0 0.0 0.0" rpy="0.0 0.0 0.0"/>
                 <geometry>
-                <box size="0.035 0.035 0.06"/>
+                <box size="0.036 0.036 0.06"/>
                 </geometry>
             </collision>
